File: kicad/halfHbridge.kicad_sch (KiCad schematic)
At the start: 10 parts, among them Q1 RH6L040BGTB1, Q2 RH6L040BGTB1, U1 L6387

Commit message: test
Parts:
- R4: footprint Resistor_SMD:R_0603_1608Metric_Pad0.98x0.95mm_HandSolder -> Resistor_SMD:R_0402_1005Metric_Pad0.72x0.64mm_HandSolder
Changed lines of the file:
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@@
 			)
 		)
-		(property "Footprint" "Resistor_SMD:R_0603_1608Metric_Pad0.98x0.95mm_HandSolder"
+		(property "Footprint" "Resistor_SMD:R_0402_1005Metric_Pad0.72x0.64mm_HandSolder"
 			(at 116.84 57.658 90)
 			(effects
