File: kicad/halfHbridge.kicad_sch (KiCad schematic)
At the start: 10 parts, among them Q1 RH6L040BGTB1, Q2 RH6L040BGTB1, U1 L6387

Commit message: a
Parts:
- renumbered C1 to C4, C2 to C5, C3 to C6, Q1 to Q3, Q2 to Q4, R4 to R10, R1 to R7, R2 to R8, R3 to R9, U1 to U2
Changed lines of the file:
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@@
 		(on_board yes)
 		(dnp no)
-		(property "Reference" "#PWR01"
+		(property "Reference" "#PWR02"
 			(at 92.71 80.01 0)
 			(effects
@@
 					(unit 1)
 				)
-				(path "/643a74e6-da9a-4f0e-bb82-8f2ac15e39e7/c7e7597f-e80e-4b08-94bb-e83c44551dab/28902d94-f2ea-40ae-b377-f4b21a4213ab"
-					(reference "#PWR05")
-					(unit 1)
-				)
-				(path "/643a74e6-da9a-4f0e-bb82-8f2ac15e39e7/c7e7597f-e80e-4b08-94bb-e83c44551dab/2d9f4ec9-b352-4bcb-b522-ddb55595a624"
-					(reference "#PWR01")
-					(unit 1)
-				)
 				(path "/643a74e6-da9a-4f0e-bb82-8f2ac15e39e7/c7e7597f-e80e-4b08-94bb-e83c44551dab/7a2a0d8a-1dc1-41bd-a666-95bb60a1f8e9"
 					(reference "#PWR02")
-					(unit 1)
-				)
-				(path "/643a74e6-da9a-4f0e-bb82-8f2ac15e39e7/c7e7597f-e80e-4b08-94bb-e83c44551dab/b4beff9c-7fa6-43aa-aab0-cae274fa03e7"
-					(reference "#PWR08")
 					(unit 1)
 				)
@@
 		(dnp no)
 		(fields_autoplaced yes)
-		(property "Reference" "R2"
+		(property "Reference" "R8"
 			(at 101.6 62.23 90)
 			(effects
@@
 					(unit 1)
 				)
-				(path "/643a74e6-da9a-4f0e-bb82-8f2ac15e39e7/c7e7597f-e80e-4b08-94bb-e83c44551dab/28902d94-f2ea-40ae-b377-f4b21a4213ab"
-					(reference "R12")
-					(unit 1)
-				)
-				(path "/643a74e6-da9a-4f0e-bb82-8f2ac15e39e7/c7e7597f-e80e-4b08-94bb-e83c44551dab/2d9f4ec9-b352-4bcb-b522-ddb55595a624"
-					(reference "R2")
-					(unit 1)
-				)
 				(path "/643a74e6-da9a-4f0e-bb82-8f2ac15e39e7/c7e7597f-e80e-4b08-94bb-e83c44551dab/7a2a0d8a-1dc1-41bd-a666-95bb60a1f8e9"
 					(reference "R8")
-					(unit 1)
-				)
-				(path "/643a74e6-da9a-4f0e-bb82-8f2ac15e39e7/c7e7597f-e80e-4b08-94bb-e83c44551dab/b4beff9c-7fa6-43aa-aab0-cae274fa03e7"
-					(reference "R24")
 					(unit 1)
 				)
@@
 		(dnp no)
 		(fields_autoplaced yes)
-		(property "Reference" "C1"
+		(property "Reference" "C4"
 			(at 55.88 62.2299 0)
 			(effects
@@
 					(unit 1)
 				)
-				(path "/643a74e6-da9a-4f0e-bb82-8f2ac15e39e7/c7e7597f-e80e-4b08-94bb-e83c44551dab/28902d94-f2ea-40ae-b377-f4b21a4213ab"
-					(reference "C7")
-					(unit 1)
-				)
-				(path "/643a74e6-da9a-4f0e-bb82-8f2ac15e39e7/c7e7597f-e80e-4b08-94bb-e83c44551dab/2d9f4ec9-b352-4bcb-b522-ddb55595a624"
-					(reference "C1")
-					(unit 1)
-				)
 				(path "/643a74e6-da9a-4f0e-bb82-8f2ac15e39e7/c7e7597f-e80e-4b08-94bb-e83c44551dab/7a2a0d8a-1dc1-41bd-a666-95bb60a1f8e9"
 					(reference "C4")
-					(unit 1)
-				)
-				(path "/643a74e6-da9a-4f0e-bb82-8f2ac15e39e7/c7e7597f-e80e-4b08-94bb-e83c44551dab/b4beff9c-7fa6-43aa-aab0-cae274fa03e7"
-					(reference "C16")
 					(unit 1)
 				)
@@
 		(dnp no)
 		(fields_autoplaced yes)
-		(property "Reference" "Q2"
+		(property "Reference" "Q4"
 			(at 127 67.3099 0)
 			(effects
@@
 					(unit 1)
 				)
-				(path "/643a74e6-da9a-4f0e-bb82-8f2ac15e39e7/c7e7597f-e80e-4b08-94bb-e83c44551dab/28902d94-f2ea-40ae-b377-f4b21a4213ab"
-					(reference "Q6")
-					(unit 1)
-				)
-				(path "/643a74e6-da9a-4f0e-bb82-8f2ac15e39e7/c7e7597f-e80e-4b08-94bb-e83c44551dab/2d9f4ec9-b352-4bcb-b522-ddb55595a624"
-					(reference "Q2")
-					(unit 1)
-				)
 				(path "/643a74e6-da9a-4f0e-bb82-8f2ac15e39e7/c7e7597f-e80e-4b08-94bb-e83c44551dab/7a2a0d8a-1dc1-41bd-a666-95bb60a1f8e9"
 					(reference "Q4")
-					(unit 1)
-				)
-				(path "/643a74e6-da9a-4f0e-bb82-8f2ac15e39e7/c7e7597f-e80e-4b08-94bb-e83c44551dab/b4beff9c-7fa6-43aa-aab0-cae274fa03e7"
-					(reference "Q12")
 					(unit 1)
 				)
@@
 		(dnp no)
 		(fields_autoplaced yes)
-		(property "Reference" "R4"
+		(property "Reference" "R10"
 			(at 116.84 49.53 90)
 			(effects
@@
 					(unit 1)
 				)
-				(path "/643a74e6-da9a-4f0e-bb82-8f2ac15e39e7/c7e7597f-e80e-4b08-94bb-e83c44551dab/28902d94-f2ea-40ae-b377-f4b21a4213ab"
-					(reference "R14")
-					(unit 1)
-				)
-				(path "/643a74e6-da9a-4f0e-bb82-8f2ac15e39e7/c7e7597f-e80e-4b08-94bb-e83c44551dab/2d9f4ec9-b352-4bcb-b522-ddb55595a624"
-					(reference "R4")
-					(unit 1)
-				)
 				(path "/643a74e6-da9a-4f0e-bb82-8f2ac15e39e7/c7e7597f-e80e-4b08-94bb-e83c44551dab/7a2a0d8a-1dc1-41bd-a666-95bb60a1f8e9"
 					(reference "R10")
-					(unit 1)
-				)
-				(path "/643a74e6-da9a-4f0e-bb82-8f2ac15e39e7/c7e7597f-e80e-4b08-94bb-e83c44551dab/b4beff9c-7fa6-43aa-aab0-cae274fa03e7"
-					(reference "R26")
 					(unit 1)
 				)
@@
 		(dnp no)
 		(fields_autoplaced yes)
-		(property "Reference" "U1"
+		(property "Reference" "U2"
 			(at 92.3133 45.72 0)
 			(effects
@@
 					(unit 1)
 				)
-				(path "/643a74e6-da9a-4f0e-bb82-8f2ac15e39e7/c7e7597f-e80e-4b08-94bb-e83c44551dab/28902d94-f2ea-40ae-b377-f4b21a4213ab"
-					(reference "U3")
-					(unit 1)
-				)
-				(path "/643a74e6-da9a-4f0e-bb82-8f2ac15e39e7/c7e7597f-e80e-4b08-94bb-e83c44551dab/2d9f4ec9-b352-4bcb-b522-ddb55595a624"
-					(reference "U1")
-					(unit 1)
-				)
 				(path "/643a74e6-da9a-4f0e-bb82-8f2ac15e39e7/c7e7597f-e80e-4b08-94bb-e83c44551dab/7a2a0d8a-1dc1-41bd-a666-95bb60a1f8e9"
 					(reference "U2")
-					(unit 1)
-				)
-				(path "/643a74e6-da9a-4f0e-bb82-8f2ac15e39e7/c7e7597f-e80e-4b08-94bb-e83c44551dab/b4beff9c-7fa6-43aa-aab0-cae274fa03e7"
-					(reference "U6")
 					(unit 1)
 				)
@@
 		(dnp no)
 		(fields_autoplaced yes)
-		(property "Reference" "C2"
+		(property "Reference" "C5"
 			(at 67.31 62.2299 0)
 			(effects
@@
 					(unit 1)
 				)
-				(path "/643a74e6-da9a-4f0e-bb82-8f2ac15e39e7/c7e7597f-e80e-4b08-94bb-e83c44551dab/28902d94-f2ea-40ae-b377-f4b21a4213ab"
-					(reference "C8")
-					(unit 1)
-				)
-				(path "/643a74e6-da9a-4f0e-bb82-8f2ac15e39e7/c7e7597f-e80e-4b08-94bb-e83c44551dab/2d9f4ec9-b352-4bcb-b522-ddb55595a624"
-					(reference "C2")
-					(unit 1)
-				)
 				(path "/643a74e6-da9a-4f0e-bb82-8f2ac15e39e7/c7e7597f-e80e-4b08-94bb-e83c44551dab/7a2a0d8a-1dc1-41bd-a666-95bb60a1f8e9"
 					(reference "C5")
-					(unit 1)
-				)
-				(path "/643a74e6-da9a-4f0e-bb82-8f2ac15e39e7/c7e7597f-e80e-4b08-94bb-e83c44551dab/b4beff9c-7fa6-43aa-aab0-cae274fa03e7"
-					(reference "C17")
 					(unit 1)
 				)
@@
 		(dnp no)
 		(fields_autoplaced yes)
-		(property "Reference" "C3"
+		(property "Reference" "C6"
 			(at 110.49 60.9599 0)
 			(effects
@@
 					(unit 1)
 				)
-				(path "/643a74e6-da9a-4f0e-bb82-8f2ac15e39e7/c7e7597f-e80e-4b08-94bb-e83c44551dab/28902d94-f2ea-40ae-b377-f4b21a4213ab"
-					(reference "C9")
-					(unit 1)
-				)
-				(path "/643a74e6-da9a-4f0e-bb82-8f2ac15e39e7/c7e7597f-e80e-4b08-94bb-e83c44551dab/2d9f4ec9-b352-4bcb-b522-ddb55595a624"
-					(reference "C3")
-					(unit 1)
-				)
 				(path "/643a74e6-da9a-4f0e-bb82-8f2ac15e39e7/c7e7597f-e80e-4b08-94bb-e83c44551dab/7a2a0d8a-1dc1-41bd-a666-95bb60a1f8e9"
 					(reference "C6")
-					(unit 1)
-				)
-				(path "/643a74e6-da9a-4f0e-bb82-8f2ac15e39e7/c7e7597f-e80e-4b08-94bb-e83c44551dab/b4beff9c-7fa6-43aa-aab0-cae274fa03e7"
-					(reference "C18")
 					(unit 1)
 				)
@@
 		(dnp no)
 		(fields_autoplaced yes)
-		(property "Reference" "R1"
+		(property "Reference" "R7"
 			(at 101.6 49.53 90)
 			(effects
@@
 					(unit 1)
 				)
-				(path "/643a74e6-da9a-4f0e-bb82-8f2ac15e39e7/c7e7597f-e80e-4b08-94bb-e83c44551dab/28902d94-f2ea-40ae-b377-f4b21a4213ab"
-					(reference "R11")
-					(unit 1)
-				)
-				(path "/643a74e6-da9a-4f0e-bb82-8f2ac15e39e7/c7e7597f-e80e-4b08-94bb-e83c44551dab/2d9f4ec9-b352-4bcb-b522-ddb55595a624"
-					(reference "R1")
-					(unit 1)
-				)
 				(path "/643a74e6-da9a-4f0e-bb82-8f2ac15e39e7/c7e7597f-e80e-4b08-94bb-e83c44551dab/7a2a0d8a-1dc1-41bd-a666-95bb60a1f8e9"
 					(reference "R7")
-					(unit 1)
-				)
-				(path "/643a74e6-da9a-4f0e-bb82-8f2ac15e39e7/c7e7597f-e80e-4b08-94bb-e83c44551dab/b4beff9c-7fa6-43aa-aab0-cae274fa03e7"
-					(reference "R23")
 					(unit 1)
 				)
@@
 		(dnp no)
 		(fields_autoplaced yes)
-		(property "Reference" "Q1"
+		(property "Reference" "Q3"
 			(at 127 49.5299 0)
 			(effects
@@
 					(unit 1)
 				)
-				(path "/643a74e6-da9a-4f0e-bb82-8f2ac15e39e7/c7e7597f-e80e-4b08-94bb-e83c44551dab/28902d94-f2ea-40ae-b377-f4b21a4213ab"
-					(reference "Q5")
-					(unit 1)
-				)
-				(path "/643a74e6-da9a-4f0e-bb82-8f2ac15e39e7/c7e7597f-e80e-4b08-94bb-e83c44551dab/2d9f4ec9-b352-4bcb-b522-ddb55595a624"
-					(reference "Q1")
-					(unit 1)
-				)
 				(path "/643a74e6-da9a-4f0e-bb82-8f2ac15e39e7/c7e7597f-e80e-4b08-94bb-e83c44551dab/7a2a0d8a-1dc1-41bd-a666-95bb60a1f8e9"
 					(reference "Q3")
-					(unit 1)
-				)
-				(path "/643a74e6-da9a-4f0e-bb82-8f2ac15e39e7/c7e7597f-e80e-4b08-94bb-e83c44551dab/b4beff9c-7fa6-43aa-aab0-cae274fa03e7"
-					(reference "Q11")
 					(unit 1)
 				)
@@
 		(dnp no)
 		(fields_autoplaced yes)
-		(property "Reference" "R3"
+		(property "Reference" "R9"
 			(at 118.11 71.1199 0)
 			(effects
@@
 					(unit 1)
 				)
-				(path "/643a74e6-da9a-4f0e-bb82-8f2ac15e39e7/c7e7597f-e80e-4b08-94bb-e83c44551dab/28902d94-f2ea-40ae-b377-f4b21a4213ab"
-					(reference "R13")
-					(unit 1)
-				)
-				(path "/643a74e6-da9a-4f0e-bb82-8f2ac15e39e7/c7e7597f-e80e-4b08-94bb-e83c44551dab/2d9f4ec9-b352-4bcb-b522-ddb55595a624"
-					(reference "R3")
-					(unit 1)
-				)
 				(path "/643a74e6-da9a-4f0e-bb82-8f2ac15e39e7/c7e7597f-e80e-4b08-94bb-e83c44551dab/7a2a0d8a-1dc1-41bd-a666-95bb60a1f8e9"
 					(reference "R9")
 					(unit 1)
 				)
-				(path "/643a74e6-da9a-4f0e-bb82-8f2ac15e39e7/c7e7597f-e80e-4b08-94bb-e83c44551dab/b4beff9c-7fa6-43aa-aab0-cae274fa03e7"
-					(reference "R25")
-					(unit 1)
-				)
