File: kicad/power.kicad_sch (KiCad schematic)
At the start: 88 parts, among them J3 Conn_01x01_Pin, J9 Conn_01x02_Pin, U11 AMS1117-5.0, U12 ACS711xEXLT-15AB, U13 LM2937xMP, U15 MAX40200AUK, U7 AMS1117-3.3, U8 ACS711xEXLT-15AB, U9 ACS711xEXLT-15AB

Commit message: test
Parts:
- removed C31, C50, C51, C52, C53, C54, C55, C56, C57: 22uF, Capacitor_SMD:C_0603_1608Metric, symbol Device:C
- C24: value 22uF -> 470u; footprint Capacitor_SMD:C_0603_1608Metric -> Capacitor_SMD:C_Elec_10x10.2
- J9: footprint Connector_AMASS:AMASS_XT30PW-M_1x02_P2.50mm_Horizontal -> Connector_AMASS:AMASS_XT30U-M_1x02_P5.0mm_Vertical
Connections:
- net +3.3V: no longer R48.1, R49.1, R54.1
- net VREF: now also R48.1, R49.1, R54.1
