File: kicad/power.kicad_sch (KiCad schematic)
At the start: 88 parts, among them J3 Conn_01x01_Pin, J9 Conn_01x02_Pin, U11 AMS1117-5.0, U12 ACS711xEXLT-15AB, U13 LM2937xMP, U15 MAX40200AUK, U7 AMS1117-3.3, U8 ACS711xEXLT-15AB, U9 ACS711xEXLT-15AB

Commit message: test
Parts:
- removed C19, C20, C22: 10u, Capacitor_SMD:C_0603_1608Metric, symbol Device:C
- removed C21, C33, C34, C35, C36, C37: 1u, Capacitor_SMD:C_0402_1005Metric, symbol Device:C
- removed C24, C31, C40, C41, C42, C43, C44, C45, C46, C47, C48, C49, C50, C51, C52, C53, C54, C55, C56, C57: 22uF, Capacitor_SMD:C_0603_1608Metric, symbol Device:C
- removed C25, C29: 10uF, Capacitor_SMD:C_0603_1608Metric, symbol Device:C
- removed C26, C28, C30: 22uF, Capacitor_SMD:C_0805_2012Metric, symbol Device:C
- removed C27: 0.47uF, Capacitor_SMD:C_0603_1608Metric, symbol Device:C
- removed C32, C38, C59, C61, C63: 0.1u, Capacitor_SMD:C_0402_1005Metric, symbol Device:C
- removed C58, C60, C62: 100u, Capacitor_SMD:C_0603_1608Metric, symbol Device:C
- removed D1, D3: 1N5819WS, Diode_SMD:D_SOD-323, symbol Diode:1N5819WS
- removed D13, D15, D16, D17: LED, LED_SMD:LED_0603_1608Metric, symbol Device:LED
- removed J3: Conn_01x01_Pin, Connector_PinHeader_2.54mm:PinHeader_1x01_P2.54mm_Vertical, symbol Connector:Conn_01x01_Pin
- removed J9: Conn_01x02_Pin, Connector_AMASS:AMASS_XT30PW-M_1x02_P2.50mm_Horizontal, symbol Connector:Conn_01x02_Pin
- removed L1, L3: L, Inductor_SMD:L_0603_1608Metric_Pad1.05x0.95mm_HandSolder, symbol Device:L
- removed R44, R45, R51: 5m, Resistor_SMD:R_2010_5025Metric_Pad1.40x2.65mm_HandSolder, symbol Device:R
- removed R46, R47, R52: 1.5k, Resistor_SMD:R_0402_1005Metric_Pad0.72x0.64mm_HandSolder, symbol Device:R
- removed R48, R49, R54: 68k, Resistor_SMD:R_0402_1005Metric_Pad0.72x0.64mm_HandSolder, symbol Device:R
- removed R50, R53, R55, R59: 2.2k, Resistor_SMD:R_0402_1005Metric_Pad0.72x0.64mm_HandSolder, symbol Device:R
- removed R56: 22k, Resistor_SMD:R_0402_1005Metric_Pad0.72x0.64mm_HandSolder, symbol Device:R
- removed R57: 10k, Resistor_SMD:R_0402_1005Metric_Pad0.72x0.64mm_HandSolder, symbol Device:R
- removed R58: 4.7k, Resistor_SMD:R_0402_1005Metric_Pad0.72x0.64mm_HandSolder, symbol Device:R
- removed TP1, TP10, TP11, TP12, TP2, TP3, TP4, TP5, TP6, TP7, TP8, TP9: TestPoint, TestPoint:TestPoint_Pad_D1.0mm, symbol Connector:TestPoint
- removed U11: AMS1117-5.0, Package_TO_SOT_SMD:SOT-223-3_TabPin2, symbol Regulator_Linear:AMS1117-5.0
- removed U12, U8, U9: ACS711xEXLT-15AB, Sensor_Current:Allegro_QFN-12-10-1EP_3x3mm_P0.5mm, symbol Sensor_Current:ACS711xEXLT-15AB
- removed U13: LM2937xMP, Package_TO_SOT_SMD:SOT-223-3_TabPin2, symbol Regulator_Linear:LM2937xMP
- removed U15: MAX40200AUK, Package_TO_SOT_SMD:SOT-23-5, symbol Analog_Switch:MAX40200AUK
- removed U7: AMS1117-3.3, Package_TO_SOT_SMD:SOT-223-3_TabPin2, symbol Regulator_Linear:AMS1117-3.3
Other:
- removed sheet halfHbridge4
- removed sheet halfHbridge5
- removed sheet halfHbridge6
- removed sheet halfHbridge7
- removed sheet halfHbridge8
- removed sheet halfHbridge9
- note removed: "パワー回路"
- note removed: "電源回路"
