File: kicad/ESC_v3.kicad_pcb (KiCad board)
At the start: 6 copper layers, 50 x 50 mm, 164 parts, among them J1 Conn_01x05_Pin, J2 Conn_01x05_Pin, J4 Conn_01x06_Pin, J6 Conn_01x06_Pin, J7 Conn_01x02_Pin, J8 Conn_01x04_Pin, J9 Conn_01x02_Pin, Q1 RH6L040BGTB1, Q10 RH6L040BGTB1, Q11 RH6L040BGTB1, Q12 RH6L040BGTB1, Q2 RH6L040BGTB1, Q3 RH6L040BGTB1, Q4 RH6L040BGTB1, Q5 RH6L040BGTB1, Q6 RH6L040BGTB1, Q7 RH6L040BGTB1, Q8 RH6L040BGTB1, Q9 RH6L040BGTB1, SW2 SW_Nidec_CAS-120A1, U1 L6387, U10 BD4104, U11 AMS1117-5.0, U12 ACS711xEXLT-15AB, U13 LM2937xMP, U14 MCP9700x-ETT, U15 MAX40200AUK, U16 AS5048A, U19 STM32G431CBUx, U2 L6387, U3 L6387, U4 L6387, U5 L6387, U6 L6387, U7 AMS1117-3.3, U8 ACS711xEXLT-15AB, U9 ACS711xEXLT-15AB

Commit message: circuit finish
Routing:
- net GND: track 108.5 -> 128.8 mm, vias 194 -> 209
- net +3.3V: track 63.6 -> 75.2 mm
- net TIM2_CH1: track 26.2 -> 22.8 mm
- net button: track 25.9 -> 28.5 mm
- net TIM4_CH2: track 63.3 -> 60.8 mm
- net TIM8_CH2: track 36.5 -> 34.9 mm
- net ADC1_IN11: track 40.3 -> 39.5 mm, vias 4 -> 3
- net VCC: vias 119 -> 145
