File: kicad/ESC_v3.kicad_pcb (KiCad board)
At the start: 4 copper layers, 50 x 50 mm, 175 parts, among them J1 Conn_01x05_Pin, J2 Conn_01x05_Pin, J3 Conn_01x01_Pin, J4 Conn_01x06_Pin, J5 Conn_01x02_Pin, J6 Conn_01x06_Pin, J7 Conn_01x02_Pin, J8 Conn_01x04_Pin, J9 Conn_01x02_Pin, Q1 RH6L040BGTB1, Q10 RH6L040BGTB1, Q11 RH6L040BGTB1, Q12 RH6L040BGTB1, Q2 RH6L040BGTB1, Q3 RH6L040BGTB1, Q4 RH6L040BGTB1, Q5 RH6L040BGTB1, Q6 RH6L040BGTB1, Q7 RH6L040BGTB1, Q8 RH6L040BGTB1, Q9 RH6L040BGTB1, SW2 SW_Nidec_CAS-120A1, U1 L6387, U10 BD4104, U11 AMS1117-5.0, U12 ACS711xEXLT-15AB, U13 LM2937xMP, U14 MCP9700x-ETT, U15 MAX40200AUK, U19 STM32G431CBUx, U2 L6387, U3 L6387, U4 L6387, U5 L6387, U6 L6387, U7 AMS1117-3.3, U8 ACS711xEXLT-15AB, U9 ACS711xEXLT-15AB

Commit message: test
Parts:
- removed BZ1: Buzzer, jisaku:buzzer_unified
- removed C31, C45, C46, C47, C48, C49, C50, C51, C52, C53, C54, C55, C56, C57: 22uF, Capacitor_SMD:C_0603_1608Metric
- removed J3: Conn_01x01_Pin, Connector_PinHeader_2.54mm:PinHeader_1x01_P2.54mm_Vertical
- removed J5: Conn_01x02_Pin, Connector_PinHeader_2.54mm:PinHeader_1x02_P2.54mm_Vertical
- removed R29: 100, Resistor_SMD:R_0402_1005Metric_Pad0.72x0.64mm_HandSolder
- removed REF** (x4): ToolingHole_1.152mm, MountingHole:ToolingHole_1.152mm
- added C39: 0.1u, Capacitor_SMD:C_0402_1005Metric, F.Cu at (87.9, 90.1)
- added H1: MountingHole, MountingHole:MountingHole_3.2mm_M3, F.Cu at (53.5, 53.5)
- added H2: MountingHole, MountingHole:MountingHole_3.2mm_M3, F.Cu at (53.5, 96.5)
- added H3: MountingHole, MountingHole:MountingHole_3.2mm_M3, F.Cu at (96.5, 53.5)
- added H4: MountingHole, MountingHole:MountingHole_3.2mm_M3, F.Cu at (96.5, 96.5)
- added R5: 10k, Resistor_SMD:R_0402_1005Metric_Pad0.72x0.64mm_HandSolder, F.Cu at (87.9, 92.1)
- added TP13: TestPoint, TestPoint:TestPoint_Pad_1.0x1.0mm, F.Cu at (54.7, 91.5)
- added TP14: TestPoint, TestPoint:TestPoint_Pad_1.0x1.0mm, F.Cu at (52.7, 91.5)
- added TP15: TestPoint, TestPoint:TestPoint_Pad_1.0x1.0mm, F.Cu at (58.0, 97.4)
- added U16: AS5048A, Package_SO:TSSOP-14_4.4x5mm_P0.65mm, B.Cu at (84.8, 71.0)
- added button1: SW_Push, Button_Switch_SMD:SW_SPST_PTS810, F.Cu at (84.6, 91.3)
- C24: value 22uF -> 470u; footprint Capacitor_SMD:C_0603_1608Metric -> Capacitor_SMD:C_Elec_10x10.2
- J1, J2: footprint Connector_JST:JST_XH_S5B-XH-A_1x05_P2.50mm_Horizontal -> Connector_JST:JST_XH_B5B-XH-A_1x05_P2.50mm_Vertical; moved to F.Cu
- J4, J8, SW2: moved to F.Cu
- J7: footprint Connector_JST:JST_XH_S2B-XH-A_1x02_P2.50mm_Horizontal -> Connector_JST:JST_XH_B2B-XH-A_1x02_P2.50mm_Vertical; moved to F.Cu
- J9: footprint Connector_AMASS:AMASS_XT30PW-M_1x02_P2.50mm_Horizontal -> Connector_AMASS:AMASS_XT30U-M_1x02_P5.0mm_Vertical
- R10, R14, R18, R22, R26, R4: footprint Resistor_SMD:R_0603_1608Metric_Pad0.98x0.95mm_HandSolder -> Resistor_SMD:R_0402_1005Metric_Pad0.72x0.64mm_HandSolder; moved to F.Cu
- moved G*** 48.2 mm to (125.6, 94.1)
- moved G*** 48.2 mm to (120.5, 90.3)
- moved G*** 48.2 mm to (119.9, 96.5)
- moved G*** 48.2 mm to (117.1, 90.4)
- moved C30 47.8 mm to (91.1, 80.9), turned to 180 degrees
- moved SW2 46.9 mm to (98.3, 83.7)
- moved D13 46.0 mm to (91.2, 70.0), turned to 180 degrees
- moved C29 44.1 mm to (81.5, 87.7)
- moved D3 44.0 mm to (83.1, 87.6)
- moved U7 43.5 mm to (88.5, 85.5)
- moved R59 43.5 mm to (97.7, 92.5)
- moved R56 41.9 mm to (90.0, 71.9), turned to -90 degrees
- moved J8 41.1 mm to (94.7, 83.8), turned to 0 degrees
- moved D17 40.9 mm to (92.1, 90.7), turned to -90 degrees
- moved C37 40.6 mm to (69.3, 99.0), turned to -90 degrees
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Connections:
- R48 pad 1: +3.3V -> VREF
- R49 pad 1: +3.3V -> VREF
- R54 pad 1: +3.3V -> VREF
Routing:
- net GND: track 228.4 -> 108.5 mm, vias 340 -> 194
- net +5V: track 75.3 -> 177.9 mm, vias 104 -> 17
- net +3.3V: track 152.6 -> 63.6 mm, vias 94 -> 28
- net +12V: track 56.0 -> 139.7 mm, vias 53 -> 14
- net EXTI13: track 2.83 -> 62.1 mm, vias 0 -> 1
- net SPI1_SCK: track 8.97 -> 68.2 mm, vias 0 -> 3
- net SS: track 26.3 -> 85.2 mm, vias 2 -> 4
- net TIM3_CH1: track 7.64 -> 65.2 mm, vias 1 -> 4
- net TIM3_CH2: track 2.73 -> 59.0 mm, vias 0 -> 1
- net SPI1_MISO: track 10.2 -> 64.4 mm, vias 1 -> 3
- net SPI1_MOSI: track 12.1 -> 62.2 mm, vias 1 -> 2
- net TIM4_CH2: track 16.9 -> 63.3 mm
- net ADC2_IN10: track 66.5 -> 25.1 mm, vias 8 -> 4
- net TIM1_CH1: track 23.2 -> 58.9 mm
- net TIM1_CH3: track 9.81 -> 44.9 mm, vias 0 -> 2
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- added copper zone on In3.Cu, net +12V
- added copper zone on In3.Cu, net +3.3V
- added copper zone on In3.Cu, net +5V
- added copper zone on In3.Cu, net /POWER/halfHbridge4/GND_mech
- added copper zone on In4.Cu, net /POWER/halfHbridge4/GND_mech
- added copper zone on In3.Cu, net /POWER/halfHbridge4/out1
- added copper zone on In4.Cu, net /POWER/halfHbridge4/out1
- added copper zone on In3.Cu, net /POWER/halfHbridge5/GND_mech
- added copper zone on In4.Cu, net /POWER/halfHbridge5/GND_mech
- added copper zone on In3.Cu, net /POWER/halfHbridge5/out1
- added copper zone on In4.Cu, net /POWER/halfHbridge5/out1
- added copper zone on In3.Cu, net /POWER/halfHbridge6/GND_mech
- added copper zone on In4.Cu, net /POWER/halfHbridge6/GND_mech
- added copper zone on In3.Cu, net /POWER/halfHbridge6/out1
- added copper zone on In4.Cu, net /POWER/halfHbridge6/out1
- added copper zone on In3.Cu, net /POWER/halfHbridge7/GND_mech
- added copper zone on In4.Cu, net /POWER/halfHbridge7/GND_mech
- added copper zone on In3.Cu, net /POWER/halfHbridge7/out1
- added copper zone on In4.Cu, net /POWER/halfHbridge7/out1
- added copper zone on In3.Cu, net /POWER/halfHbridge8/GND_mech
- added copper zone on In4.Cu, net /POWER/halfHbridge8/GND_mech
- added copper zone on In3.Cu, net /POWER/halfHbridge8/out1
- added copper zone on In4.Cu, net /POWER/halfHbridge8/out1
- added copper zone on In3.Cu, net /POWER/halfHbridge9/GND_mech
- added copper zone on In4.Cu, net /POWER/halfHbridge9/GND_mech
- added copper zone on In3.Cu, net /POWER/halfHbridge9/out1
- added copper zone on In4.Cu, net /POWER/halfHbridge9/out1
- added copper zone on In3.Cu, net GND
- added copper zone on In4.Cu, net GND
- added copper zone on In3.Cu, net VCC
- added copper zone on In4.Cu, net VCC
- removed copper zone on In1.Cu, net +12V
- removed copper zone on In1.Cu, net +3.3V
- removed copper zone on In1.Cu, net +5V
Other:
- copper layers 4 -> 6
- board text removed: "18~3.3"
- board text removed: "3.3V"
- board text removed: "5V"
- board text removed: "A"
- board text removed: "AMP1"
- board text removed: "AMP2"
- board text removed: "AMP3"
- board text removed: "B"
- board text removed: "C/Z"
- board text removed: "CLK"
- board text removed: "DIO"
- board text removed: "G"
- board text removed: "GND"
- board text removed: "H"
- board text removed: "H/L"
- board text removed: "L"
- board text removed: "L/H"
- board text removed: "MISO"
- board text removed: "MOSI"
- board text removed: "NRST"
- board text removed: "RX"
- board text removed: "SCK"
- board text removed: "SCL"
- board text removed: "SDA"
- board text removed: "SS"
- board text removed: "TIM1 CH3/2/1"
- board text removed: "TIM8 CH3/2/1"
- board text removed: "TX"
- board text removed: "VI"
- board text removed: "VO"

Commit message: final
Parts:
- added G***: LOGO, LOGO, B.Cu at (56.3, 58.9)
- moved G*** 70.6 mm to (56.1, 81.3), turned to 180 degrees
- moved G*** 64.3 mm to (56.4, 86.6), turned to 180 degrees
- moved G*** 64.2 mm to (56.4, 91.9), turned to 180 degrees
- moved G*** 60.8 mm to (56.5, 95.4), turned to 180 degrees
Connections:
- J6 pad 1: +3.3V -> RX
- J6 pad 2: DIO -> TX
- J6 pad 3: CLK -> GND
- J6 pad 4: GND -> CLK
- J6 pad 5: TX -> DIO
- J6 pad 6: RX -> +3.3V
Routing:
- net TX: track 40.7 -> 59.1 mm
- net CLK: track 42.9 -> 33.3 mm, vias 1 -> 2
- net DIO: track 45.0 -> 36.2 mm, vias 3 -> 1
- net OPAMP2_VINP: track 64.8 -> 72.5 mm, vias 4 -> 3
- net ToggleSwitch: track 37.2 -> 44.7 mm
- net RX: track 39.6 -> 46.7 mm
- net CAN_L: track 22.1 -> 16.6 mm
- net TIM2_CH1: track 26.2 -> 21.9 mm
- net +3.3V: track 63.6 -> 67.3 mm, vias 28 -> 27
- net TIM8_CH2: track 36.5 -> 33.6 mm
- net CAN_TX: track 13.9 -> 16.2 mm, vias 3 -> 2
- net ADC2_IN10: track 25.1 -> 23.5 mm
- net TIM4_CH2: track 63.3 -> 64.9 mm
- net +5V: track 177.9 -> 179.3 mm
- net OPAMP1_VINP: track 54.4 -> 55.7 mm
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Other:
- board text added: "1"
- board text added: "120Ω"
- board text added: "2"
- board text added: "3"
- board text added: "3V"
- board text added: "5V"
- board text added: "CL"
- board text added: "CLK"
- board text added: "DIO"
- board text added: "G"
- board text added: "H"
- board text added: "L"
- board text added: "RST"
- board text added: "RX"
- board text added: "SCL"
- board text added: "SDA"
- board text added: "SS"
- board text added: "TX"

Commit message: a
Connections:
- U16 pad 11: unconnected-(U16-VDD5V-Pad11) -> +3.3V
- U16 pad 13: unconnected-(U16-GND-Pad13) -> GND
- U16 pad 5: unconnected-(U16-TEST-Pad5) -> GND
Routing:
- net GND: track 107.2 -> 114.4 mm
- net +3.3V: track 67.3 -> 68.0 mm
Changed lines of the file:
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@@
 	(net 118 "unconnected-(U10-SPLIT-Pad5)")
 	(net 119 "unconnected-(U16-TEST-Pad10)")
-	(net 120 "unconnected-(U16-GND-Pad13)")
-	(net 121 "unconnected-(U16-TEST-Pad7)")
-	(net 122 "unconnected-(U16-PWM-Pad14)")
-	(net 123 "unconnected-(U16-VDD5V-Pad11)")
-	(net 124 "unconnected-(U16-TEST-Pad6)")
-	(net 125 "unconnected-(U16-TEST-Pad8)")
-	(net 126 "unconnected-(U16-TEST-Pad5)")
-	(net 127 "unconnected-(U16-TEST-Pad9)")
-	(net 128 "Net-(R43-Pad2)")
+	(net 120 "unconnected-(U16-TEST-Pad7)")
+	(net 121 "unconnected-(U16-PWM-Pad14)")
+	(net 122 "unconnected-(U16-TEST-Pad6)")
+	(net 123 "unconnected-(U16-TEST-Pad8)")
+	(net 124 "unconnected-(U16-TEST-Pad9)")
+	(net 125 "Net-(R43-Pad2)")
 	(footprint "Resistor_SMD:R_2010_5025Metric_Pad1.40x2.65mm_HandSolder"
 		(layer "F.Cu")
@@
 			(size 1 1)
 			(layers "F.Cu" "F.Mask")
-			(net 128 "Net-(R43-Pad2)")
+			(net 125 "Net-(R43-Pad2)")
 			(pinfunction "1")
 			(pintype "passive")
@@
 			(layers "F.Cu" "F.Mask" "F.Paste")
 			(roundrect_rratio 0.25)
-			(net 128 "Net-(R43-Pad2)")
+			(net 125 "Net-(R43-Pad2)")
 			(pintype "passive")
 		)
@@
 			(layers "B.Cu" "B.Mask" "B.Paste")
 			(roundrect_rratio 0.25)
-			(net 126 "unconnected-(U16-TEST-Pad5)")
+			(net 107 "GND")
 			(pinfunction "TEST")
 			(pintype "passive")
@@
 			(layers "B.Cu" "B.Mask" "B.Paste")
 			(roundrect_rratio 0.25)
-			(net 124 "unconnected-(U16-TEST-Pad6)")
+			(net 122 "unconnected-(U16-TEST-Pad6)")
 			(pinfunction "TEST")
 			(pintype "passive")
@@
 			(layers "B.Cu" "B.Mask" "B.Paste")
 			(roundrect_rratio 0.25)
-			(net 121 "unconnected-(U16-TEST-Pad7)")
+			(net 120 "unconnected-(U16-TEST-Pad7)")
 			(pinfunction "TEST")
 			(pintype "passive")
@@
 			(layers "B.Cu" "B.Mask" "B.Paste")
 			(roundrect_rratio 0.25)
-			(net 125 "unconnected-(U16-TEST-Pad8)")
+			(net 123 "unconnected-(U16-TEST-Pad8)")
 			(pinfunction "TEST")
 			(pintype "passive")
@@
 			(layers "B.Cu" "B.Mask" "B.Paste")
 			(roundrect_rratio 0.25)
-			(net 127 "unconnected-(U16-TEST-Pad9)")
+			(net 124 "unconnected-(U16-TEST-Pad9)")
 			(pinfunction "TEST")
 			(pintype "passive")
@@
 			(layers "B.Cu" "B.Mask" "B.Paste")
 			(roundrect_rratio 0.25)
-			(net 123 "unconnected-(U16-VDD5V-Pad11)")
+			(net 12 "+3.3V")
 			(pinfunction "VDD5V")
 			(pintype "power_in")
@@
 			(layers "B.Cu" "B.Mask" "B.Paste")
 			(roundrect_rratio 0.25)
-			(net 120 "unconnected-(U16-GND-Pad13)")
+			(net 107 "GND")
 			(pinfunction "GND")
 			(pintype "power_in")
@@
 			(layers "B.Cu" "B.Mask" "B.Paste")
 			(roundrect_rratio 0.25)
-			(net 122 "unconnected-(U16-PWM-Pad14)")
+			(net 121 "unconnected-(U16-PWM-Pad14)")
 			(pinfunction "PWM")
 			(pintype "output")
@@
 	)
 	(segment
+		(start 84.7852 73.8555)
+		(end 84.1352 73.8555)
+		(width 0.2)
+		(layer "B.Cu")
+		(net 12)
+	)
+	(segment
 		(start 84.1352 78.928)
 		(end 84.1352 80.3252)
@@
 	)
 	(segment
+		(start 83.4852 73.8555)
+		(end 83.4852 73.087898)
+		(width 0.2)
+		(layer "B.Cu")
+		(net 107)
+	)
+	(segment
 		(start 81.534 83.9484)
 		(end 81.534 81.293)
@@
 	)
 	(segment
+		(start 83.721305 72.851793)
+		(end 83.721305 71.083524)
+		(width 0.2)
+		(layer "B.Cu")
+		(net 107)
+	)
+	(segment
 		(start 87.5857 80.8671)
 		(end 87.0432 80.3246)
@@
 	)
 	(segment
+		(start 85.4352 68.867999)
+		(end 83.678699 70.6245)
+		(width 0.2)
+		(layer "B.Cu")
+		(net 107)
+	)
+	(segment
 		(start 81.534 81.293)
 		(end 81.4578 81.2168)
@@
 	)
 	(segment
+		(start 83.4852 73.087898)
+		(end 83.721305 72.851793)
+		(width 0.2)
+		(layer "B.Cu")
+		(net 107)
+	)
+	(segment
 		(start 55.6862 68.4396)
 		(end 54.628519 68.4396)
@@
 	)
 	(segment
+		(start 83.678699 70.6245)
+		(end 83.262281 70.6245)
+		(width 0.2)
+		(layer "B.Cu")
+		(net 107)
+	)
+	(segment
 		(start 87.0432 80.3246)
 		(end 87.0432 78.2831)
@@
 	)
 	(segment
+		(start 85.4352 68.1305)
+		(end 85.4352 68.867999)
+		(width 0.2)
+		(layer "B.Cu")
+		(net 107)
+	)
+	(segment
+		(start 83.721305 71.083524)
+		(end 83.262281 70.6245)
+		(width 0.2)
+		(layer "B.Cu")
+		(net 107)
+	)
+	(segment
 		(start 71.2242 98.311639)
 		(end 71.2242 97.6969)
@@
 		(width 0.2)
 		(layer "F.Cu")
-		(net 128)
+		(net 125)
 	)
 	(segment
@@
 		(width 0.2)
 		(layer "F.Cu")
-		(net 128)
+		(net 125)
 	)
 	(zone
