File: kicad/spk.kicad_sch (KiCad schematic)
At the start: 11 parts, among them U15 LM386

Commit message: a
Parts:
- RV1: footprint (none) -> Potentiometer_THT:Potentiometer_ACP_CA9-H3,8_Horizontal
Changed lines of the file:
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@@
 			)
 		)
-		(property "Footprint" ""
+		(property "Footprint" "Potentiometer_THT:Potentiometer_ACP_CA9-H3,8_Horizontal"
 			(at 102.87 55.88 0)
 			(effects
