File: kicad/power_stage.kicad_sch (KiCad schematic)
At the start: 6 parts, among them Q4 RH6L040BGTB1, Q5 RH6L040BGTB1

Commit message: a
Connections:
- net OPAMP_P: now reaches Q5.1 (S), R8.1
Changed lines of the file:
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@@
+		)
+	)
+	(hierarchical_label "OPAMP_P"
+		(shape input)
+		(at 114.3 83.82 0)
+		(effects
+			(font
+				(size 1.27 1.27)
+			)
+			(justify left)
 		)
 	)
@@
 		(shape input)
 		(at 114.3 73.66 0)
+		(effects
+			(font
+				(size 1.27 1.27)
+			)
+			(justify left)
+		)
+	)
+	(hierarchical_label "OPAMP_M"
+		(shape input)
+		(at 114.3 91.44 0)
 		(effects
 			(font
@@
 					(unit 1)
 				)
+				(path "/643a74e6-da9a-4f0e-bb82-8f2ac15e39e7/b58b0be8-8252-4a19-bb00-8315ea20fe3c"
+					(reference "R?")
+					(unit 1)
+				)
 				(path "/643a74e6-da9a-4f0e-bb82-8f2ac15e39e7/f6007c1e-2115-4cff-923c-cb43600cb7fd"
 					(reference "R11")
@@
 					(unit 1)
 				)
+				(path "/643a74e6-da9a-4f0e-bb82-8f2ac15e39e7/b58b0be8-8252-4a19-bb00-8315ea20fe3c"
+					(reference "C?")
+					(unit 1)
+				)

Commit message: a
Parts:
- C2: value C -> 1u; footprint (none) -> Capacitor_SMD:C_0402_1005Metric
- R1, R7: footprint (none) -> Resistor_SMD:R_0402_1005Metric_Pad0.72x0.64mm_HandSolder
- R8: footprint (none) -> Resistor_SMD:R_2010_5025Metric
Changed lines of the file:
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@@
 			)
 		)
-		(property "Footprint" ""
+		(property "Footprint" "Resistor_SMD:R_0402_1005Metric_Pad0.72x0.64mm_HandSolder"
 			(at 96.52 70.358 90)
 			(effects
@@
 			)
 		)
-		(property "Footprint" ""
+		(property "Footprint" "Resistor_SMD:R_2010_5025Metric"
 			(at 112.522 87.63 90)
 			(effects
@@
 				)
 				(path "/643a74e6-da9a-4f0e-bb82-8f2ac15e39e7/b58b0be8-8252-4a19-bb00-8315ea20fe3c"
-					(reference "R?")
+					(reference "R18")
 					(unit 1)
 				)
@@
 			)
 		)
-		(property "Footprint" ""
+		(property "Footprint" "Resistor_SMD:R_0402_1005Metric_Pad0.72x0.64mm_HandSolder"
 			(at 96.52 80.518 90)
 			(effects
@@
 			)
 		)
-		(property "Value" "C"
+		(property "Value" "1u"
 			(at 106.68 69.8499 0)
 			(effects
@@
 			)
 		)
-		(property "Footprint" ""
+		(property "Footprint" "Capacitor_SMD:C_0402_1005Metric"
 			(at 103.8352 72.39 0)
 			(effects
@@
 				)
 				(path "/643a74e6-da9a-4f0e-bb82-8f2ac15e39e7/b58b0be8-8252-4a19-bb00-8315ea20fe3c"
-					(reference "C?")
-					(unit 1)
-				)
+					(reference "C5")
+					(unit 1)
+				)

Commit message: a
Parts:
- removed R8: R, Resistor_SMD:R_2010_5025Metric, symbol Device:R
Connections:
- net OPAMP_P is gone; now on net GND: Q5.1 (S)
Changed lines of the file:
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@@
 	(wire
 		(pts
-			(xy 114.3 91.44) (xy 114.3 93.98)
+			(xy 114.3 83.82) (xy 114.3 93.98)
 		)
 		(stroke
@@
 		)
 	)
-	(hierarchical_label "OPAMP_P"
-		(shape input)
-		(at 114.3 83.82 0)
-		(effects
-			(font
-				(size 1.27 1.27)
-			)
-			(justify left)
-		)
-	)
 	(hierarchical_label "OUT"
 		(shape input)
@@
 		(shape input)
 		(at 114.3 73.66 0)
-		(effects
-			(font
-				(size 1.27 1.27)
-			)
-			(justify left)
-		)
-	)
-	(hierarchical_label "OPAMP_M"
-		(shape input)
-		(at 114.3 91.44 0)
 		(effects
 			(font
@@
 					(unit 1)
 				)
-			)
-		)
-	)
-	(symbol
-		(lib_id "Device:R")
-		(at 114.3 87.63 0)
-		(unit 1)
-		(exclude_from_sim no)
-		(in_bom yes)
-		(on_board yes)
-		(dnp no)
-		(fields_autoplaced yes)
-		(property "Reference" "R8"
-			(at 116.84 86.3599 0)
-			(effects
-				(font
-					(size 1.27 1.27)
-				)
-				(justify left)
-			)
-		)
-		(property "Value" "R"
-			(at 116.84 88.8999 0)
-			(effects
-				(font
-					(size 1.27 1.27)
-				)
-				(justify left)
-			)
-		)
-		(property "Footprint" "Resistor_SMD:R_2010_5025Metric"
-			(at 112.522 87.63 90)
-			(effects
-				(font
-					(size 1.27 1.27)
-				)
-				(hide yes)
-			)
-		)
-		(property "Datasheet" "~"
-			(at 114.3 87.63 0)
-			(effects
-				(font
-					(size 1.27 1.27)
-				)
-				(hide yes)
-			)
-		)
-		(property "Description" "Resistor"
-			(at 114.3 87.63 0)
-			(effects
-				(font
-					(size 1.27 1.27)
-				)
-				(hide yes)
-			)
-		)
-		(pin "2"
-		)
-		(pin "1"
-		)
-		(instances
-			(project "ESC_v3"
-				(path "/643a74e6-da9a-4f0e-bb82-8f2ac15e39e7/89dab747-500c-4d30-aaae-2892da5dc15f"
-					(reference "R8")
-					(unit 1)
-				)
-				(path "/643a74e6-da9a-4f0e-bb82-8f2ac15e39e7/b58b0be8-8252-4a19-bb00-8315ea20fe3c"
-					(reference "R18")
-					(unit 1)
-				)
-				(path "/643a74e6-da9a-4f0e-bb82-8f2ac15e39e7/f6007c1e-2115-4cff-923c-cb43600cb7fd"
-					(reference "R11")
-					(unit 1)
-				)

Commit message: order finished
Parts:
- R1, R7: value R -> 10
Changed lines of the file:
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@@
 			)
 		)
-		(property "Value" "R"
+		(property "Value" "10"
 			(at 96.52 64.77 90)
 			(effects
@@
 			)
 		)
-		(property "Value" "R"
+		(property "Value" "10"
 			(at 96.52 74.93 90)
 			(effects
