File: kicad/ESC_v3.kicad_sch (KiCad schematic)
At the start: 79 parts, among them J1 Conn_01x07, J10 Conn_01x03, J2 Conn_01x05_Pin, J3 USB_C_Receptacle_USB2.0, J4 Conn_01x04, J6 Conn_01x06_Pin, J7 Conn_01x02_Pin, J8 Conn_01x04_Pin, J9 Conn_01x02, SW2 SW_Nidec_CAS-120A1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

Commit message: add v2_mini_mini
Parts:
- removed D3: 1N5819WS, Diode_SMD:D_SOD-323_HandSoldering, symbol Diode:1N4148WT
- removed J3: USB_C_Receptacle_USB2.0, Connector_USB:USB_C_Receptacle_GCT_USB4105-xx-A_16P_TopMnt_Horizontal, symbol Connector:USB_C_Receptacle_USB2.0
- removed J8: Conn_01x04_Pin, Connector_PinSocket_2.54mm:PinSocket_1x04_P2.54mm_Vertical, symbol Connector:Conn_01x04_Pin
- removed R23, R24: 5.1k, Resistor_SMD:R_0603_1608Metric, symbol Device:R
- added D13: LED_R, LED_SMD:LED_0603_1608Metric, symbol Device:LED
- added R35: 10k, Resistor_SMD:R_0402_1005Metric_Pad0.72x0.64mm_HandSolder, symbol Device:R
- J7: footprint Connector_JST:JST_XH_B2B-XH-A_1x02_P2.50mm_Vertical -> jisaku:名称未設定_1
Connections:
- net +3.3V: no longer R13.2
- net +5V: now also TP1.1
- net GND: now also R35.1; no longer C10.2, C9.2, J9.1 (Pin_1), R2.2, U1.25 (PB2), U2.1 (GND)
- net VCC: now reaches C1.1, C8.1, L1.2, U1.63 (VCC)
- net VCC: now also D13.2 (A)
- net power_stage/GND renamed power_stage2/GND
- new net: D13.1 (K), R35.2
- new net OPAMP3_VINM: C10.2, C9.2, J9.1 (Pin_1), R2.2, U1.25 (PB2), U2.1 (GND)
Other:
- moved on the sheet: D10, D11, D12, R12, R13, R14, R27, R28, R30, R8
